Commit message: gripper fix

File: robot_urdf/generated_urdf/ur5.urdf (robot description, URDF)
Before this commit: robot ur_robot, 30 links, 29 joints
Links:
- added link tavolo_link; collision box size=1 0.15 0.15; collision box size=1 0.8 0.04
Joints:
- added joint tavolo_joint: type fixed, parent base_link, child tavolo_link, origin xyz=-0.5 -0.35 -1.75 rpy=0 0 0
- joint world_joint: origin xyz=0 0 0 rpy=0 0 0 -> xyz=0.5 0.35 1.75 rpy=0 0 0
